Commit message: d

File: description/gazebo_control.xacro (robot description, xacro)
@@ -7,5 +7,5 @@
             <right_joint>right_rear_wheel</right_joint>
             <!-- [m] from SW -->
-            <wheel_seperation>0.068185</wheel_seperation>
+            <wheel_separation>0.068185</wheel_separation>
             <!-- [m] from urdf -->
             <wheel_radius>0.0815</wheel_radius>

File: description/robot.urdf.xacro (robot description, xacro)
@@ -1,9 +1,14 @@
 <?xml version="1.0"?>
 <robot xmlns:xacro="http://www.ros.org/wiki/xacro"  name="robot">
+    <xacro:arg name="use_ros2_control" default="false"/>
     <!-- URDF Robot Description-->
     <xacro:include filename="robot_core.xacro" />
-    <!-- Gazebo ros2_control plugins-->
-    <!--<xacro:include filename="gazebo_control.xacro" /> -->
-    <!-- ROS2 Control plugins-->
-    <xacro:include filename="ros2_control.xacro" />
+    <xacro:if value="$(arg use_ros2_control)">
+        <!-- ROS2 Control plugins-->
+        <xacro:include filename="ros2_control.xacro" />
+    </xacro:if>
+    <xacro:unless value="$(arg use_ros2_control)">
+        <!-- Gazebo ros2_control plugins-->
+        <xacro:include filename="gazebo_control.xacro" />
+    </xacro:unless>
 </robot>

File: description/robot_core.xacro (robot description, xacro)
@@ -82,5 +82,5 @@
   </gazebo>
   <!-- _____________DIFF TO LEFT DIFF JOINT____________-->
-  <joint name="left_diff" type="revolute"> <!--diff_to_left_diff-->
+  <joint name="left_diff" type="fixed"> <!--diff_to_left_diff-->
     <origin xyz="0 0 -0.28" rpy="-3.1416 0 -3.1416"/>
     <axis xyz="0 0 1"/>
@@ -116,5 +116,5 @@
   </gazebo>
   <!-- _____________LEFT DIFF TO LEFT REAR LIN JOINT____________-->
-  <joint name="left_rear_linear" type="prismatic"> <!-- left_diff_to_left_rear_lin -->
+  <joint name="left_rear_linear" type="fixed"> <!-- left_diff_to_left_rear_lin -->
     <limit effort="1000.0" lower="0" upper="0.13" velocity="0.5"/>
     <origin xyz="-0.216 -0.0010724 0" rpy="-1.5708 0 0.0049647"/>
@@ -179,5 +179,5 @@
   </gazebo>
     <!-- _____________LEFT DIFF TO LEFT FRONT LIN JOINT____________-->
-  <joint name="left_front_linear" type="prismatic"> <!-- left_diff_to_left_front_lin-->
+  <joint name="left_front_linear" type="fixed"> <!-- left_diff_to_left_front_lin-->
     <limit effort="1000.0" lower="0" upper="0.13" velocity="0.5"/>
     <origin xyz="0.216 0.0010724 0" rpy="-1.5708 0 0.0049647"/>
@@ -244,5 +244,5 @@
   </link>
     <!-- _____________DIFF TO RIGHT DIFF JOINT____________-->
-    <joint name="right_diff" type="revolute"> <!-- diff_to_right_diff -->
+    <joint name="right_diff" type="fixed"> <!-- diff_to_right_diff -->
       <origin xyz="0 0 0.28" rpy="0 0 0"/>
       <axis xyz="0 0 1"/>
@@ -279,5 +279,5 @@
     </gazebo>
     <!-- _____________RIGHT DIFF TO RIGHT REAR LIN JOINT____________-->
-    <joint name="right_rear_linear" type="prismatic"> <!-- right_diff_to_right_rear_lin -->
+    <joint name="right_rear_linear" type="fixed"> <!-- right_diff_to_right_rear_lin -->
       <limit effort="1000.0" lower="0" upper="0.13" velocity="0.5"/>
       <origin xyz="-0.216 -0.0010724 0" rpy="-1.5708 0 0.0049647"/>
@@ -342,5 +342,5 @@
     </gazebo>
       <!-- _____________RIGHT DIFF TO RIGHT FRONT LIN JOINT____________-->
-    <joint name="right_front_linear" type="prismatic"> <!-- right_diff_to_right_front_lin -->
+    <joint name="right_front_linear" type="fixed"> <!-- right_diff_to_right_front_lin -->
       <limit effort="1000.0" lower="0" upper="0.13" velocity="0.5"/>
       <origin xyz="0.216 0.0010724 0" rpy="-1.5708 0 0.0049647"/>

File: description/ros2_control.xacro (robot description, xacro)
@@ -18,4 +18,14 @@
             <state_interface name="position"></state_interface>
         </joint>
+        <joint name="left_rear_wheel">
+            <command_interface name="velocity"/>
+            <state_interface name="velocity"></state_interface>
+            <state_interface name="position"></state_interface>
+        </joint>
+        <joint name="right_rear_wheel">
+            <command_interface name="velocity"/>
+            <state_interface name="velocity"></state_interface>
+            <state_interface name="position"></state_interface>
+        </joint>
     </ros2_control>
         <!-- GZ plugin -->
