Commit message: d

File: description/ros2_control_odrive.xacro (robot description, xacro)
@@ -7,6 +7,33 @@
             <param name="can">can0</param>
         </hardware>
+        <joint name="right_rear_linear">
+            <param name="node_id">3</param>
+            <command_interface name="position"/>
+            <command_interface name="velocity"/>
+            <command_interface name="effort"/>
+            <state_interface name="position"/>
+            <state_interface name="velocity"/>
+            <state_interface name="effort"/>
+        </joint>
+        <joint name="right_front_linear">
+            <param name="node_id">2</param>
+            <command_interface name="position"/>
+            <command_interface name="velocity"/>
+            <command_interface name="effort"/>
+            <state_interface name="position"/>
+            <state_interface name="velocity"/>
+            <state_interface name="effort"/>
+        </joint>
         <joint name="left_rear_linear">
-            <param name="node_id">3</param>
+            <param name="node_id">1</param>
+            <command_interface name="position"/>
+            <command_interface name="velocity"/>
+            <command_interface name="effort"/>
+            <state_interface name="position"/>
+            <state_interface name="velocity"/>
+            <state_interface name="effort"/>
+        </joint>
+        <joint name="left_front_linear">
+            <param name="node_id">0</param>
             <command_interface name="position"/>
             <command_interface name="velocity"/>
