Commit message: lidar_gz

File: description/robot.urdf.xacro (robot description, xacro)
@@ -1,13 +1,15 @@
 <?xml version="1.0"?>
 <robot xmlns:xacro="http://www.ros.org/wiki/xacro"  name="robot">
+    <!-- Arguments -->
     <xacro:arg name="use_ros2_control" default="true"/>
     <!-- URDF Robot Description-->
     <xacro:include filename="robot_core.xacro" />
+    <!-- Sensors -->
+    <xacro:include filename="lidar.xacro" />
+    <!-- Control -->
     <xacro:if value="$(arg use_ros2_control)">
-        <!-- ROS2 Control plugins-->
         <xacro:include filename="ros2_control.xacro" />
     </xacro:if>
     <xacro:unless value="$(arg use_ros2_control)">
-        <!-- Gazebo ros2_control plugins-->
         <xacro:include filename="gazebo_control.xacro" />
     </xacro:unless>

File: description/robot_core.xacro (robot description, xacro)
@@ -6,4 +6,7 @@
 <material name="black">
   <color rgba="${64/255} ${64/255} ${64/255} 1" />
+</material>
+<material name="blue">
+  <color rgba="${0/255} ${0/255} ${255/255} 1" />
 </material>
 <material name="mesh_color">

Commit message: f

File: description/robot.urdf.xacro (robot description, xacro)
@@ -9,5 +9,5 @@
     <!-- Control -->
     <xacro:if value="$(arg use_ros2_control)">
-        <xacro:include filename="ros2_control.xacro" />
+        <xacro:include filename="ros2_control_odrive.xacro" />
     </xacro:if>
     <xacro:unless value="$(arg use_ros2_control)">

File: description/robot_core.xacro (robot description, xacro)
@@ -119,5 +119,5 @@
   </gazebo>
   <!-- _____________LEFT DIFF TO LEFT REAR LIN JOINT____________-->
-  <joint name="left_rear_linear" type="fixed"> <!-- left_diff_to_left_rear_lin -->
+  <joint name="left_rear_linear" type="prismatic"> <!-- left_diff_to_left_rear_lin -->
     <limit effort="1000.0" lower="0" upper="0.13" velocity="0.5"/>
     <origin xyz="-0.216 -0.0010724 0" rpy="-1.5708 0 0.0049647"/>

Commit message: d

File: description/robot.urdf.xacro (robot description, xacro)
@@ -10,5 +10,4 @@
     <xacro:if value="$(arg use_ros2_control)">
         <xacro:include filename="ros2_control.xacro" />
-        <xacro:include filename="ros2_control_odrive.xacro" />
     </xacro:if>
     <xacro:unless value="$(arg use_ros2_control)">

File: description/ros2_control.xacro (robot description, xacro)
@@ -21,41 +21,3 @@
         </joint>
     </ros2_control>
-    <ros2_control name="myactuator_controller_right_rear_wheel" type="actuator">
-        <hardware>
-            <plugin>myactuator_rmd_hardware/MyActuatorRmdHardwareInterface</plugin>
-            <param name="ifname">can2</param>
-            <param name="actuator_id">5</param>
-            <param name="torque_constant">2.023914969</param>
-            <param name="velocity_alpha">0.1</param>
-            <param name="effort_alpha">0.1</param>
-            <param name="cycle_time">1</param>
-        </hardware>
-        <joint name="right_rear_wheel">
-            <command_interface name="position"/>
-            <command_interface name="velocity"/>
-            <command_interface name="effort"/>
-            <state_interface name="position"/>
-            <state_interface name="velocity"/>
-            <state_interface name="effort"/>
-        </joint>
-    </ros2_control>
-    <ros2_control name="myactuator_controller_left_front_wheel" type="actuator">
-        <hardware>
-            <plugin>myactuator_rmd_hardware/MyActuatorRmdHardwareInterface</plugin>
-            <param name="ifname">can0</param>
-            <param name="actuator_id">6</param>
-            <param name="torque_constant">2.023914969</param>
-            <param name="velocity_alpha">0.1</param>
-            <param name="effort_alpha">0.1</param>
-            <param name="cycle_time">1</param>
-        </hardware>
-        <joint name="left_front_wheel">
-            <command_interface name="position"/>
-            <command_interface name="velocity"/>
-            <command_interface name="effort"/>
-            <state_interface name="position"/>
-            <state_interface name="velocity"/>
-            <state_interface name="effort"/>
-        </joint>
-    </ros2_control>
 </robot>
