Commit message: g

File: description/ros2_control.xacro (robot description, xacro)
@@ -1,4 +1,25 @@
 <?xml version="1.0"?>
 <robot xmlns:xacro="http://www.ros.org/wiki/xacro">
+    <ros2_control name="${some_name}" type="actuator">
+    <hardware>
+        <plugin>myactuator_rmd_hardware/MyActuatorRmdHardwareInterface</plugin>
+        <param name="ifname">${ifname}</param>
+        <param name="actuator_id">${actuator_id}</param>
+        <param name="torque_constant">${torque_constant}</param>
+        <!-- Optional: Low-pass filters for velocity and effort (0 < alpha <= 1); defaults to no filter -->
+        <param name="velocity_alpha">0.1</param>
+        <param name="effort_alpha">0.1</param>
+        <!-- Optional: Cycle time of the asynchronous thread; defaults to 1ms (1000Hz) -->
+        <param name="cycle_time">1</param>
+    </hardware>
+    <joint name="${joint_name}">
+        <command_interface name="position"/>
+        <command_interface name="velocity"/>
+        <command_interface name="effort"/>
+        <state_interface name="position"/>
+        <state_interface name="velocity"/>
+        <state_interface name="effort"/>
+    </joint>
+    </ros2_control>
     <!-- ROS2 Control plugin for Gazebo-->
     <ros2_control name="GazeboSystem" type="system">

Commit message: g

File: description/ros2_control.xacro (robot description, xacro)
@@ -1,10 +1,10 @@
 <?xml version="1.0"?>
 <robot xmlns:xacro="http://www.ros.org/wiki/xacro">
-    <ros2_control name="${some_name}" type="actuator">
+    <ros2_control name="myactuator_controller" type="actuator">
     <hardware>
         <plugin>myactuator_rmd_hardware/MyActuatorRmdHardwareInterface</plugin>
-        <param name="ifname">${ifname}</param>
-        <param name="actuator_id">${actuator_id}</param>
-        <param name="torque_constant">${torque_constant}</param>
+        <param name="can0">${ifname}</param>
+        <param name="actuator_id">145</param>
+        <param name="torque_constant">2.023914969</param>
         <!-- Optional: Low-pass filters for velocity and effort (0 < alpha <= 1); defaults to no filter -->
         <param name="velocity_alpha">0.1</param>
@@ -23,11 +23,11 @@
     </ros2_control>
     <!-- ROS2 Control plugin for Gazebo-->
-    <ros2_control name="GazeboSystem" type="system">
+    <!--ros2_control name="GazeboSystem" type="system"-->
         <!-- Hardware interface for GZ-->
-        <hardware>
+        <!--hardware>
             <plugin>gz_ros2_control/GazeboSimSystem</plugin>
-        </hardware>
+        </hardware-->
         <!-- All continous joints-->
-        <joint name="left_front_wheel">
+        <!--joint name="left_front_wheel">
             <command_interface name="velocity"/>
             <state_interface name="velocity"></state_interface>
@@ -49,10 +49,10 @@
             <state_interface name="position"></state_interface>
         </joint>
-    </ros2_control>
+    </ros2_control-->
         <!-- GZ plugin -->
-    <gazebo>
+    <!--gazebo>
           <plugin name="gz_ros2_control::GazeboSimROS2ControlPlugin" filename="libgz_ros2_control-system.so">
             <parameters>$(find kridtbot)/config/my_controllers.yaml</parameters>
         </plugin>
-    </gazebo>
+    </gazebo-->
 </robot>

Commit message: f

File: description/ros2_control.xacro (robot description, xacro)
@@ -4,5 +4,5 @@
     <hardware>
         <plugin>myactuator_rmd_hardware/MyActuatorRmdHardwareInterface</plugin>
-        <param name="can0">${ifname}</param>
+        <param name="ifname">can0</param>
         <param name="actuator_id">145</param>
         <param name="torque_constant">2.023914969</param>
@@ -13,5 +13,5 @@
         <param name="cycle_time">1</param>
     </hardware>
-    <joint name="${joint_name}">
+    <joint name="left_front_wheel">
         <command_interface name="position"/>
         <command_interface name="velocity"/>

Commit message: f

File: description/ros2_control.xacro (robot description, xacro)
@@ -2,57 +2,21 @@
 <robot xmlns:xacro="http://www.ros.org/wiki/xacro">
     <ros2_control name="myactuator_controller" type="actuator">
-    <hardware>
-        <plugin>myactuator_rmd_hardware/MyActuatorRmdHardwareInterface</plugin>
-        <param name="ifname">can0</param>
-        <param name="actuator_id">145</param>
-        <param name="torque_constant">2.023914969</param>
-        <!-- Optional: Low-pass filters for velocity and effort (0 < alpha <= 1); defaults to no filter -->
-        <param name="velocity_alpha">0.1</param>
-        <param name="effort_alpha">0.1</param>
-        <!-- Optional: Cycle time of the asynchronous thread; defaults to 1ms (1000Hz) -->
-        <param name="cycle_time">1</param>
-    </hardware>
-    <joint name="left_front_wheel">
-        <command_interface name="position"/>
-        <command_interface name="velocity"/>
-        <command_interface name="effort"/>
-        <state_interface name="position"/>
-        <state_interface name="velocity"/>
-        <state_interface name="effort"/>
-    </joint>
+        <hardware>
+            <plugin>myactuator_rmd_hardware/MyActuatorRmdHardwareInterface</plugin>
+            <param name="ifname">can0</param>
+            <param name="actuator_id">145</param>
+            <param name="torque_constant">2.023914969</param>
+            <param name="velocity_alpha">0.1</param>
+            <param name="effort_alpha">0.1</param>
+            <param name="cycle_time">1</param>
+        </hardware>
+        <joint name="left_front_wheel">
+            <command_interface name="position"/>
+            <command_interface name="velocity"/>
+            <command_interface name="effort"/>
+            <state_interface name="position"/>
+            <state_interface name="velocity"/>
+            <state_interface name="effort"/>
+        </joint>
     </ros2_control>
-    <!-- ROS2 Control plugin for Gazebo-->
-    <!--ros2_control name="GazeboSystem" type="system"-->
-        <!-- Hardware interface for GZ-->
-        <!--hardware>
-            <plugin>gz_ros2_control/GazeboSimSystem</plugin>
-        </hardware-->
-        <!-- All continous joints-->
-        <!--joint name="left_front_wheel">
-            <command_interface name="velocity"/>
-            <state_interface name="velocity"></state_interface>
-            <state_interface name="position"></state_interface>
-        </joint>
-        <joint name="right_front_wheel">
-            <command_interface name="velocity"/>
-            <state_interface name="velocity"></state_interface>
-            <state_interface name="position"></state_interface>
-        </joint>
-        <joint name="left_rear_wheel">
-            <command_interface name="velocity"/>
-            <state_interface name="velocity"></state_interface>
-            <state_interface name="position"></state_interface>
-        </joint>
-        <joint name="right_rear_wheel">
-            <command_interface name="velocity"/>
-            <state_interface name="velocity"></state_interface>
-            <state_interface name="position"></state_interface>
-        </joint>
-    </ros2_control-->
-        <!-- GZ plugin -->
-    <!--gazebo>
-          <plugin name="gz_ros2_control::GazeboSimROS2ControlPlugin" filename="libgz_ros2_control-system.so">
-            <parameters>$(find kridtbot)/config/my_controllers.yaml</parameters>
-        </plugin>
-    </gazebo-->
 </robot>

Commit message: w

File: description/ros2_control.xacro (robot description, xacro)
@@ -1,22 +1,37 @@
 <?xml version="1.0"?>
 <robot xmlns:xacro="http://www.ros.org/wiki/xacro">
-    <ros2_control name="myactuator_controller" type="actuator">
+    <!-- ROS2 Control plugin for Gazebo-->
+    <ros2_control name="GazeboSystem" type="system">
+        <!-- Hardware interface for GZ-->
         <hardware>
-            <plugin>myactuator_rmd_hardware/MyActuatorRmdHardwareInterface</plugin>
-            <param name="ifname">can0</param>
-            <param name="actuator_id">6</param>
-            <param name="torque_constant">2.023914969</param>
-            <param name="velocity_alpha">0.1</param>
-            <param name="effort_alpha">0.1</param>
-            <param name="cycle_time">1</param>
+            <plugin>gz_ros2_control/GazeboSimSystem</plugin>
         </hardware>
+        <!-- All continous joints-->
         <joint name="left_front_wheel">
-            <command_interface name="position"/>
             <command_interface name="velocity"/>
-            <command_interface name="effort"/>
-            <state_interface name="position"/>
-            <state_interface name="velocity"/>
-            <state_interface name="effort"/>
+            <state_interface name="velocity"></state_interface>
+            <state_interface name="position"></state_interface>
+        </joint>
+        <joint name="right_front_wheel">
+            <command_interface name="velocity"/>
+            <state_interface name="velocity"></state_interface>
+            <state_interface name="position"></state_interface>
+        </joint>
+        <joint name="left_rear_wheel">
+            <command_interface name="velocity"/>
+            <state_interface name="velocity"></state_interface>
+            <state_interface name="position"></state_interface>
+        </joint>
+        <joint name="right_rear_wheel">
+            <command_interface name="velocity"/>
+            <state_interface name="velocity"></state_interface>
+            <state_interface name="position"></state_interface>
         </joint>
     </ros2_control>
+        <!-- GZ plugin -->
+    <gazebo>
+          <plugin name="gz_ros2_control::GazeboSimROS2ControlPlugin" filename="libgz_ros2_control-system.so">
+            <parameters>$(find kridtbot)/config/my_controllers.yaml</parameters>
+        </plugin>
+    </gazebo>
 </robot>

Commit message: d

File: description/ros2_control.xacro (robot description, xacro)
@@ -2,36 +2,22 @@
 <robot xmlns:xacro="http://www.ros.org/wiki/xacro">
     <!-- ROS2 Control plugin for Gazebo-->
-    <ros2_control name="GazeboSystem" type="system">
-        <!-- Hardware interface for GZ-->
+    <ros2_control name="myactuator_controller" type="actuator">
         <hardware>
-            <plugin>gz_ros2_control/GazeboSimSystem</plugin>
+            <plugin>myactuator_rmd_hardware/MyActuatorRmdHardwareInterface</plugin>
+            <param name="ifname">can0</param>
+            <param name="actuator_id">6</param>
+            <param name="torque_constant">2.023914969</param>
+            <param name="velocity_alpha">0.1</param>
+            <param name="effort_alpha">0.1</param>
+            <param name="cycle_time">1</param>
         </hardware>
-        <!-- All continous joints-->
         <joint name="left_front_wheel">
+            <command_interface name="position"/>
             <command_interface name="velocity"/>
-            <state_interface name="velocity"></state_interface>
-            <state_interface name="position"></state_interface>
-        </joint>
-        <joint name="right_front_wheel">
-            <command_interface name="velocity"/>
-            <state_interface name="velocity"></state_interface>
-            <state_interface name="position"></state_interface>
-        </joint>
-        <joint name="left_rear_wheel">
-            <command_interface name="velocity"/>
-            <state_interface name="velocity"></state_interface>
-            <state_interface name="position"></state_interface>
-        </joint>
-        <joint name="right_rear_wheel">
-            <command_interface name="velocity"/>
-            <state_interface name="velocity"></state_interface>
-            <state_interface name="position"></state_interface>
+            <command_interface name="effort"/>
+            <state_interface name="position"/>
+            <state_interface name="velocity"/>
+            <state_interface name="effort"/>
         </joint>
     </ros2_control>
-        <!-- GZ plugin -->
-    <gazebo>
-          <plugin name="gz_ros2_control::GazeboSimROS2ControlPlugin" filename="libgz_ros2_control-system.so">
-            <parameters>$(find kridtbot)/config/my_controllers.yaml</parameters>
-        </plugin>
-    </gazebo>
 </robot>

Commit message: d

File: description/ros2_control.xacro (robot description, xacro)
@@ -7,4 +7,42 @@
             <param name="ifname">can0</param>
             <param name="actuator_id">4</param>
+            <param name="torque_constant">2.023914969</param>
+            <param name="velocity_alpha">0.1</param>
+            <param name="effort_alpha">0.1</param>
+            <param name="cycle_time">1</param>
+        </hardware>
+        <joint name="right_front_wheel">
+            <command_interface name="position"/>
+            <command_interface name="velocity"/>
+            <command_interface name="effort"/>
+            <state_interface name="position"/>
+            <state_interface name="velocity"/>
+            <state_interface name="effort"/>
+        </joint>
+    </ros2_control>
+    <ros2_control name="myactuator_controller" type="actuator">
+        <hardware>
+            <plugin>myactuator_rmd_hardware/MyActuatorRmdHardwareInterface</plugin>
+            <param name="ifname">can0</param>
+            <param name="actuator_id">5</param>
+            <param name="torque_constant">2.023914969</param>
+            <param name="velocity_alpha">0.1</param>
+            <param name="effort_alpha">0.1</param>
+            <param name="cycle_time">1</param>
+        </hardware>
+        <joint name="right_rear_wheel">
+            <command_interface name="position"/>
+            <command_interface name="velocity"/>
+            <command_interface name="effort"/>
+            <state_interface name="position"/>
+            <state_interface name="velocity"/>
+            <state_interface name="effort"/>
+        </joint>
+    </ros2_control>
+    <ros2_control name="myactuator_controller" type="actuator">
+        <hardware>
+            <plugin>myactuator_rmd_hardware/MyActuatorRmdHardwareInterface</plugin>
+            <param name="ifname">can0</param>
+            <param name="actuator_id">6</param>
             <param name="torque_constant">2.023914969</param>
             <param name="velocity_alpha">0.1</param>

Commit message: d

File: description/ros2_control.xacro (robot description, xacro)
@@ -21,41 +21,3 @@
         </joint>
     </ros2_control>
-    <ros2_control name="myactuator_controller_right_rear_wheel" type="actuator">
-        <hardware>
-            <plugin>myactuator_rmd_hardware/MyActuatorRmdHardwareInterface</plugin>
-            <param name="ifname">can0</param>
-            <param name="actuator_id">5</param>
-            <param name="torque_constant">2.023914969</param>
-            <param name="velocity_alpha">0.1</param>
-            <param name="effort_alpha">0.1</param>
-            <param name="cycle_time">1</param>
-        </hardware>
-        <joint name="right_rear_wheel">
-            <command_interface name="position"/>
-            <command_interface name="velocity"/>
-            <command_interface name="effort"/>
-            <state_interface name="position"/>
-            <state_interface name="velocity"/>
-            <state_interface name="effort"/>
-        </joint>
-    </ros2_control>
-    <ros2_control name="myactuator_controller_left_front_wheel" type="actuator">
-        <hardware>
-            <plugin>myactuator_rmd_hardware/MyActuatorRmdHardwareInterface</plugin>
-            <param name="ifname">can0</param>
-            <param name="actuator_id">6</param>
-            <param name="torque_constant">2.023914969</param>
-            <param name="velocity_alpha">0.1</param>
-            <param name="effort_alpha">0.1</param>
-            <param name="cycle_time">1</param>
-        </hardware>
-        <joint name="left_front_wheel">
-            <command_interface name="position"/>
-            <command_interface name="velocity"/>
-            <command_interface name="effort"/>
-            <state_interface name="position"/>
-            <state_interface name="velocity"/>
-            <state_interface name="effort"/>
-        </joint>
-    </ros2_control>
 </robot>

File: description/werwerewer.xacro (robot description, xacro)
@@ -1,5 +1,43 @@
 <?xml version="1.0"?>
 <robot xmlns:xacro="http://www.ros.org/wiki/xacro">
-    <ros2_control name="myactuator_controller" type="actuator">
+    <ros2_control name="myactuator_controller_right_front_wheel" type="actuator">
+        <hardware>
+            <plugin>myactuator_rmd_hardware/MyActuatorRmdHardwareInterface</plugin>
+            <param name="ifname">can0</param>
+            <param name="actuator_id">4</param>
+            <param name="torque_constant">2.023914969</param>
+            <param name="velocity_alpha">0.1</param>
+            <param name="effort_alpha">0.1</param>
+            <param name="cycle_time">1</param>
+        </hardware>
+        <joint name="right_front_wheel">
+            <command_interface name="position"/>
+            <command_interface name="velocity"/>
+            <command_interface name="effort"/>
+            <state_interface name="position"/>
+            <state_interface name="velocity"/>
+            <state_interface name="effort"/>
+        </joint>
+    </ros2_control>
+    <ros2_control name="myactuator_controller_right_rear_wheel" type="actuator">
+        <hardware>
+            <plugin>myactuator_rmd_hardware/MyActuatorRmdHardwareInterface</plugin>
+            <param name="ifname">can0</param>
+            <param name="actuator_id">5</param>
+            <param name="torque_constant">2.023914969</param>
+            <param name="velocity_alpha">0.1</param>
+            <param name="effort_alpha">0.1</param>
+            <param name="cycle_time">1</param>
+        </hardware>
+        <joint name="right_rear_wheel">
+            <command_interface name="position"/>
+            <command_interface name="velocity"/>
+            <command_interface name="effort"/>
+            <state_interface name="position"/>
+            <state_interface name="velocity"/>
+            <state_interface name="effort"/>
+        </joint>
+    </ros2_control>
+    <ros2_control name="myactuator_controller_left_front_wheel" type="actuator">
         <hardware>
             <plugin>myactuator_rmd_hardware/MyActuatorRmdHardwareInterface</plugin>

Commit message: w

File: description/ros2_control.xacro (robot description, xacro)
@@ -2,4 +2,23 @@
 <robot xmlns:xacro="http://www.ros.org/wiki/xacro">
     <!-- ROS2 Control plugin for Gazebo-->
+    <ros2_control name="myactuator_controller_left_front_wheel" type="actuator">
+        <hardware>
+            <plugin>myactuator_rmd_hardware/MyActuatorRmdHardwareInterface</plugin>
+            <param name="ifname">can0</param>
+            <param name="actuator_id">5</param>
+            <param name="torque_constant">2.023914969</param>
+            <param name="velocity_alpha">0.1</param>
+            <param name="effort_alpha">0.1</param>
+            <param name="cycle_time">1</param>
+        </hardware>
+        <joint name="left_front_wheel">
+            <command_interface name="position"/>
+            <command_interface name="velocity"/>
+            <command_interface name="effort"/>
+            <state_interface name="position"/>
+            <state_interface name="velocity"/>
+            <state_interface name="effort"/>
+        </joint>
+    </ros2_control>
     <ros2_control name="myactuator_controller_right_front_wheel" type="actuator">
         <hardware>

Commit message: d

File: description/ros2_control.xacro (robot description, xacro)
@@ -6,5 +6,5 @@
             <plugin>myactuator_rmd_hardware/MyActuatorRmdHardwareInterface</plugin>
             <param name="ifname">can0</param>
-            <param name="actuator_id">5</param>
+            <param name="actuator_id">4</param>
             <param name="torque_constant">2.023914969</param>
             <param name="velocity_alpha">0.1</param>
@@ -25,5 +25,5 @@
             <plugin>myactuator_rmd_hardware/MyActuatorRmdHardwareInterface</plugin>
             <param name="ifname">can0</param>
-            <param name="actuator_id">4</param>
+            <param name="actuator_id">5</param>
             <param name="torque_constant">2.023914969</param>
             <param name="velocity_alpha">0.1</param>
@@ -31,5 +31,5 @@
             <param name="cycle_time">1</param>
         </hardware>
-        <joint name="right_front_wheel">
+        <joint name="left_rear_wheel">
             <command_interface name="position"/>
             <command_interface name="velocity"/>

Commit message: d

File: description/ros2_control.xacro (robot description, xacro)
@@ -25,5 +25,5 @@
             <plugin>myactuator_rmd_hardware/MyActuatorRmdHardwareInterface</plugin>
             <param name="ifname">can0</param>
-            <param name="actuator_id">5</param>
+            <param name="actuator_id">6</param>
             <param name="torque_constant">2.023914969</param>
             <param name="velocity_alpha">0.1</param>
@@ -31,5 +31,5 @@
             <param name="cycle_time">1</param>
         </hardware>
-        <joint name="left_rear_wheel">
+        <joint name="right_front_wheel">
             <command_interface name="position"/>
             <command_interface name="velocity"/>
