Commit message: d

File: description/ros2_control.xacro (robot description, xacro)
@@ -21,5 +21,24 @@
         </joint>
     </ros2_control>
-    <ros2_control name="myactuator_controller_right_front_wheel" type="actuator">
+    <ros2_control name="myactuator_controller_right_rear_wheel" type="actuator">
+        <hardware>
+            <plugin>myactuator_rmd_hardware/MyActuatorRmdHardwareInterface</plugin>
+            <param name="ifname">can0</param>
+            <param name="actuator_id">5</param>
+            <param name="torque_constant">2.023914969</param>
+            <param name="velocity_alpha">0.1</param>
+            <param name="effort_alpha">0.1</param>
+            <param name="cycle_time">1</param>
+        </hardware>
+        <joint name="right_rear_wheel">
+            <command_interface name="position"/>
+            <command_interface name="velocity"/>
+            <command_interface name="effort"/>
+            <state_interface name="position"/>
+            <state_interface name="velocity"/>
+            <state_interface name="effort"/>
+        </joint>
+    </ros2_control>
+    <ros2_control name="myactuator_controller_left_front_wheel" type="actuator">
         <hardware>
             <plugin>myactuator_rmd_hardware/MyActuatorRmdHardwareInterface</plugin>
@@ -31,5 +50,24 @@
             <param name="cycle_time">1</param>
         </hardware>
-        <joint name="right_front_wheel">
+        <joint name="left_front_wheel">
+            <command_interface name="position"/>
+            <command_interface name="velocity"/>
+            <command_interface name="effort"/>
+            <state_interface name="position"/>
+            <state_interface name="velocity"/>
+            <state_interface name="effort"/>
+        </joint>
+    </ros2_control>
+    <ros2_control name="myactuator_controller_left_rear_wheel" type="actuator">
+        <hardware>
+            <plugin>myactuator_rmd_hardware/MyActuatorRmdHardwareInterface</plugin>
+            <param name="ifname">can0</param>
+            <param name="actuator_id">7</param>
+            <param name="torque_constant">2.023914969</param>
+            <param name="velocity_alpha">0.1</param>
+            <param name="effort_alpha">0.1</param>
+            <param name="cycle_time">1</param>
+        </hardware>
+        <joint name="left_rear_wheel">
             <command_interface name="position"/>
             <command_interface name="velocity"/>

Commit message: d

File: description/ros2_control.xacro (robot description, xacro)
@@ -2,42 +2,4 @@
 <robot xmlns:xacro="http://www.ros.org/wiki/xacro">
     <!-- ROS2 Control plugin for Gazebo-->
-    <ros2_control name="myactuator_controller_left_front_wheel" type="actuator">
-        <hardware>
-            <plugin>myactuator_rmd_hardware/MyActuatorRmdHardwareInterface</plugin>
-            <param name="ifname">can0</param>
-            <param name="actuator_id">4</param>
-            <param name="torque_constant">2.023914969</param>
-            <param name="velocity_alpha">0.1</param>
-            <param name="effort_alpha">0.1</param>
-            <param name="cycle_time">1</param>
-        </hardware>
-        <joint name="left_front_wheel">
-            <command_interface name="position"/>
-            <command_interface name="velocity"/>
-            <command_interface name="effort"/>
-            <state_interface name="position"/>
-            <state_interface name="velocity"/>
-            <state_interface name="effort"/>
-        </joint>
-    </ros2_control>
-    <ros2_control name="myactuator_controller_right_rear_wheel" type="actuator">
-        <hardware>
-            <plugin>myactuator_rmd_hardware/MyActuatorRmdHardwareInterface</plugin>
-            <param name="ifname">can0</param>
-            <param name="actuator_id">5</param>
-            <param name="torque_constant">2.023914969</param>
-            <param name="velocity_alpha">0.1</param>
-            <param name="effort_alpha">0.1</param>
-            <param name="cycle_time">1</param>
-        </hardware>
-        <joint name="right_rear_wheel">
-            <command_interface name="position"/>
-            <command_interface name="velocity"/>
-            <command_interface name="effort"/>
-            <state_interface name="position"/>
-            <state_interface name="velocity"/>
-            <state_interface name="effort"/>
-        </joint>
-    </ros2_control>
     <ros2_control name="myactuator_controller_left_front_wheel" type="actuator">
         <hardware>
@@ -59,22 +21,3 @@
         </joint>
     </ros2_control>
-    <ros2_control name="myactuator_controller_left_rear_wheel" type="actuator">
-        <hardware>
-            <plugin>myactuator_rmd_hardware/MyActuatorRmdHardwareInterface</plugin>
-            <param name="ifname">can0</param>
-            <param name="actuator_id">7</param>
-            <param name="torque_constant">2.023914969</param>
-            <param name="velocity_alpha">0.1</param>
-            <param name="effort_alpha">0.1</param>
-            <param name="cycle_time">1</param>
-        </hardware>
-        <joint name="left_rear_wheel">
-            <command_interface name="position"/>
-            <command_interface name="velocity"/>
-            <command_interface name="effort"/>
-            <state_interface name="position"/>
-            <state_interface name="velocity"/>
-            <state_interface name="effort"/>
-        </joint>
-    </ros2_control>
 </robot>

Commit message: d

File: description/ros2_control.xacro (robot description, xacro)
@@ -2,4 +2,42 @@
 <robot xmlns:xacro="http://www.ros.org/wiki/xacro">
     <!-- ROS2 Control plugin for Gazebo-->
+    <ros2_control name="myactuator_controller_right_front_wheel" type="actuator">
+        <hardware>
+            <plugin>myactuator_rmd_hardware/MyActuatorRmdHardwareInterface</plugin>
+            <param name="ifname">can0</param>
+            <param name="actuator_id">4</param>
+            <param name="torque_constant">2.023914969</param>
+            <param name="velocity_alpha">0.1</param>
+            <param name="effort_alpha">0.1</param>
+            <param name="cycle_time">1</param>
+        </hardware>
+        <joint name="right_front_wheel">
+            <command_interface name="position"/>
+            <command_interface name="velocity"/>
+            <command_interface name="effort"/>
+            <state_interface name="position"/>
+            <state_interface name="velocity"/>
+            <state_interface name="effort"/>
+        </joint>
+    </ros2_control>
+    <ros2_control name="myactuator_controller_right_rear_wheel" type="actuator">
+        <hardware>
+            <plugin>myactuator_rmd_hardware/MyActuatorRmdHardwareInterface</plugin>
+            <param name="ifname">can0</param>
+            <param name="actuator_id">5</param>
+            <param name="torque_constant">2.023914969</param>
+            <param name="velocity_alpha">0.1</param>
+            <param name="effort_alpha">0.1</param>
+            <param name="cycle_time">1</param>
+        </hardware>
+        <joint name="right_rear_wheel">
+            <command_interface name="position"/>
+            <command_interface name="velocity"/>
+            <command_interface name="effort"/>
+            <state_interface name="position"/>
+            <state_interface name="velocity"/>
+            <state_interface name="effort"/>
+        </joint>
+    </ros2_control>
     <ros2_control name="myactuator_controller_left_front_wheel" type="actuator">
         <hardware>

Commit message: d

File: description/ros2_control.xacro (robot description, xacro)
@@ -2,23 +2,4 @@
 <robot xmlns:xacro="http://www.ros.org/wiki/xacro">
     <!-- ROS2 Control plugin for Gazebo-->
-    <ros2_control name="myactuator_controller_right_front_wheel" type="actuator">
-        <hardware>
-            <plugin>myactuator_rmd_hardware/MyActuatorRmdHardwareInterface</plugin>
-            <param name="ifname">can0</param>
-            <param name="actuator_id">4</param>
-            <param name="torque_constant">2.023914969</param>
-            <param name="velocity_alpha">0.1</param>
-            <param name="effort_alpha">0.1</param>
-            <param name="cycle_time">1</param>
-        </hardware>
-        <joint name="right_front_wheel">
-            <command_interface name="position"/>
-            <command_interface name="velocity"/>
-            <command_interface name="effort"/>
-            <state_interface name="position"/>
-            <state_interface name="velocity"/>
-            <state_interface name="effort"/>
-        </joint>
-    </ros2_control>
     <ros2_control name="myactuator_controller_right_rear_wheel" type="actuator">
         <hardware>

Commit message: d

File: description/ros2_control.xacro (robot description, xacro)
@@ -21,22 +21,3 @@
         </joint>
     </ros2_control>
-    <ros2_control name="myactuator_controller_left_front_wheel" type="actuator">
-        <hardware>
-            <plugin>myactuator_rmd_hardware/MyActuatorRmdHardwareInterface</plugin>
-            <param name="ifname">can0</param>
-            <param name="actuator_id">6</param>
-            <param name="torque_constant">2.023914969</param>
-            <param name="velocity_alpha">0.1</param>
-            <param name="effort_alpha">0.1</param>
-            <param name="cycle_time">1</param>
-        </hardware>
-        <joint name="left_front_wheel">
-            <command_interface name="position"/>
-            <command_interface name="velocity"/>
-            <command_interface name="effort"/>
-            <state_interface name="position"/>
-            <state_interface name="velocity"/>
-            <state_interface name="effort"/>
-        </joint>
-    </ros2_control>
 </robot>

Commit message: d

File: description/ros2_control.xacro (robot description, xacro)
@@ -21,3 +21,22 @@
         </joint>
     </ros2_control>
+        <ros2_control name="myactuator_controller_right_front_wheel" type="actuator">
+        <hardware>
+            <plugin>myactuator_rmd_hardware/MyActuatorRmdHardwareInterface</plugin>
+            <param name="ifname">can0</param>
+            <param name="actuator_id">4</param>
+            <param name="torque_constant">2.023914969</param>
+            <param name="velocity_alpha">0.1</param>
+            <param name="effort_alpha">0.1</param>
+            <param name="cycle_time">1</param>
+        </hardware>
+        <joint name="right_front_wheel">
+            <command_interface name="position"/>
+            <command_interface name="velocity"/>
+            <command_interface name="effort"/>
+            <state_interface name="position"/>
+            <state_interface name="velocity"/>
+            <state_interface name="effort"/>
+        </joint>
+    </ros2_control>
 </robot>

Commit message: f

File: description/ros2_control.xacro (robot description, xacro)
@@ -2,9 +2,9 @@
 <robot xmlns:xacro="http://www.ros.org/wiki/xacro">
     <!-- ROS2 Control plugin for Gazebo-->
-    <ros2_control name="myactuator_controller_right_rear_wheel" type="actuator">
+    <ros2_control name="myactuator_controller_left_front_wheel" type="actuator">
         <hardware>
             <plugin>myactuator_rmd_hardware/MyActuatorRmdHardwareInterface</plugin>
             <param name="ifname">can0</param>
-            <param name="actuator_id">5</param>
+            <param name="actuator_id">6</param>
             <param name="torque_constant">2.023914969</param>
             <param name="velocity_alpha">0.1</param>
@@ -12,24 +12,5 @@
             <param name="cycle_time">1</param>
         </hardware>
-        <joint name="right_rear_wheel">
-            <command_interface name="position"/>
-            <command_interface name="velocity"/>
-            <command_interface name="effort"/>
-            <state_interface name="position"/>
-            <state_interface name="velocity"/>
-            <state_interface name="effort"/>
-        </joint>
-    </ros2_control>
-        <ros2_control name="myactuator_controller_right_front_wheel" type="actuator">
-        <hardware>
-            <plugin>myactuator_rmd_hardware/MyActuatorRmdHardwareInterface</plugin>
-            <param name="ifname">can0</param>
-            <param name="actuator_id">4</param>
-            <param name="torque_constant">2.023914969</param>
-            <param name="velocity_alpha">0.1</param>
-            <param name="effort_alpha">0.1</param>
-            <param name="cycle_time">1</param>
-        </hardware>
-        <joint name="right_front_wheel">
+        <joint name="left_front_wheel">
             <command_interface name="position"/>
             <command_interface name="velocity"/>

Commit message: f

File: description/ros2_control.xacro (robot description, xacro)
@@ -2,4 +2,23 @@
 <robot xmlns:xacro="http://www.ros.org/wiki/xacro">
     <!-- ROS2 Control plugin for Gazebo-->
+    <ros2_control name="myactuator_controller_right_front_wheel" type="actuator">
+        <hardware>
+            <plugin>myactuator_rmd_hardware/MyActuatorRmdHardwareInterface</plugin>
+            <param name="ifname">can1</param>
+            <param name="actuator_id">4</param>
+            <param name="torque_constant">2.023914969</param>
+            <param name="velocity_alpha">0.1</param>
+            <param name="effort_alpha">0.1</param>
+            <param name="cycle_time">1</param>
+        </hardware>
+        <joint name="right_front_wheel">
+            <command_interface name="position"/>
+            <command_interface name="velocity"/>
+            <command_interface name="effort"/>
+            <state_interface name="position"/>
+            <state_interface name="velocity"/>
+            <state_interface name="effort"/>
+        </joint>
+    </ros2_control>
     <ros2_control name="myactuator_controller_left_front_wheel" type="actuator">
         <hardware>

Commit message: d

File: description/ros2_control.xacro (robot description, xacro)
@@ -13,4 +13,23 @@
         </hardware>
         <joint name="right_front_wheel">
+            <command_interface name="position"/>
+            <command_interface name="velocity"/>
+            <command_interface name="effort"/>
+            <state_interface name="position"/>
+            <state_interface name="velocity"/>
+            <state_interface name="effort"/>
+        </joint>
+    </ros2_control>
+    <ros2_control name="myactuator_controller_right_rear_wheel" type="actuator">
+        <hardware>
+            <plugin>myactuator_rmd_hardware/MyActuatorRmdHardwareInterface</plugin>
+            <param name="ifname">can2</param>
+            <param name="actuator_id">5</param>
+            <param name="torque_constant">2.023914969</param>
+            <param name="velocity_alpha">0.1</param>
+            <param name="effort_alpha">0.1</param>
+            <param name="cycle_time">1</param>
+        </hardware>
+        <joint name="right_rear_wheel">
             <command_interface name="position"/>
             <command_interface name="velocity"/>

Commit message: d

File: description/ros2_control.xacro (robot description, xacro)
@@ -2,5 +2,24 @@
 <robot xmlns:xacro="http://www.ros.org/wiki/xacro">
     <!-- ROS2 Control plugin for Gazebo-->
-    <ros2_control name="myactuator_controller_right_front_wheel" type="actuator">
+    <ros2_control name="myactuator_controller_left_front_wheel" type="actuator">
+        <hardware>
+            <plugin>myactuator_rmd_hardware/MyActuatorRmdHardwareInterface</plugin>
+            <param name="ifname">can2</param>
+            <param name="actuator_id">6</param>
+            <param name="torque_constant">2.023914969</param>
+            <param name="velocity_alpha">0.1</param>
+            <param name="effort_alpha">0.1</param>
+            <param name="cycle_time">1</param>
+        </hardware>
+        <joint name="left_front_wheel">
+            <command_interface name="position"/>
+            <command_interface name="velocity"/>
+            <command_interface name="effort"/>
+            <state_interface name="position"/>
+            <state_interface name="velocity"/>
+            <state_interface name="effort"/>
+        </joint>
+    </ros2_control>
+    <ros2_control name="myactuator_controller_left_rear_wheel" type="actuator">
         <hardware>
             <plugin>myactuator_rmd_hardware/MyActuatorRmdHardwareInterface</plugin>
@@ -12,5 +31,5 @@
             <param name="cycle_time">1</param>
         </hardware>
-        <joint name="right_front_wheel">
+        <joint name="left_rear_wheel">
             <command_interface name="position"/>
             <command_interface name="velocity"/>

Commit message: d

File: description/ros2_control.xacro (robot description, xacro)
@@ -2,4 +2,23 @@
 <robot xmlns:xacro="http://www.ros.org/wiki/xacro">
     <!-- ROS2 Control plugin for Gazebo-->
+    <ros2_control name="myactuator_controller_right_rear_wheel" type="actuator">
+        <hardware>
+            <plugin>myactuator_rmd_hardware/MyActuatorRmdHardwareInterface</plugin>
+            <param name="ifname">can0</param>
+            <param name="actuator_id">5</param>
+            <param name="torque_constant">2.023914969</param>
+            <param name="velocity_alpha">0.1</param>
+            <param name="effort_alpha">0.1</param>
+            <param name="cycle_time">1</param>
+        </hardware>
+        <joint name="right_rear_wheel">
+            <command_interface name="position"/>
+            <command_interface name="velocity"/>
+            <command_interface name="effort"/>
+            <state_interface name="position"/>
+            <state_interface name="velocity"/>
+            <state_interface name="effort"/>
+        </joint>
+    </ros2_control>
     <ros2_control name="myactuator_controller_right_front_wheel" type="actuator">
         <hardware>
