Commit message: d

File: description/robot_core_sim.xacro (robot description, xacro)
@@ -148,5 +148,5 @@
   </gazebo>
   <!-- _____________LEFT DIFF TO LEFT REAR LIN JOINT____________-->
-  <joint name="left_rear_linear" type="prismatic"> <!-- left_diff_to_left_rear_lin -->
+  <joint name="left_rear_linear" type="fixed"> <!-- left_diff_to_left_rear_lin -->
     <!--<limit effort="1000.0" lower="0" upper="0.13" velocity="0.5"/> -->
     <origin xyz="-0.216 -0.0010724 0" rpy="-1.5708 0 0.0049647"/>
@@ -230,5 +230,5 @@
   </gazebo>
     <!-- _____________LEFT DIFF TO LEFT FRONT LIN JOINT____________-->
-  <joint name="left_front_linear" type="prismatic"> <!-- left_diff_to_left_front_lin-->
+  <joint name="left_front_linear" type="fixed"> <!-- left_diff_to_left_front_lin-->
     <!--<limit effort="1000.0" lower="0" upper="0.13" velocity="0.5"/> -->
     <origin xyz="0.216 0.0010724 0" rpy="-1.5708 0 0.0049647"/>
@@ -349,5 +349,5 @@
     </gazebo>
     <!-- _____________RIGHT DIFF TO RIGHT REAR LIN JOINT____________-->
-    <joint name="right_rear_linear" type="prismatic"> <!-- right_diff_to_right_rear_lin -->
+    <joint name="right_rear_linear" type="fixed"> <!-- right_diff_to_right_rear_lin -->
       <!--<limit effort="1000.0" lower="0" upper="0.13" velocity="0.5"/> -->
       <origin xyz="0.216 -0.0010724 0" rpy="-1.5708 0 0.0049647"/>
@@ -433,5 +433,5 @@
     </gazebo>
       <!-- _____________RIGHT DIFF TO RIGHT FRONT LIN JOINT____________-->
-    <joint name="right_front_linear" type="prismatic"> <!-- right_diff_to_right_front_lin -->
+    <joint name="right_front_linear" type="fixed"> <!-- right_diff_to_right_front_lin -->
       <!--<limit effort="1000.0" lower="0" upper="0.13" velocity="0.5"/> -->
       <origin xyz="-0.216 0.0010724 0" rpy="-1.5708 0 0.0049647"/>

File: description/robot_sim.urdf.xacro (robot description, xacro)
@@ -4,5 +4,5 @@
     <xacro:arg name="use_ros2_control" default="true"/>
     <!-- URDF Robot Description-->
-    <xacro:include filename="robot_core.xacro" />
+    <xacro:include filename="robot_core_sim.xacro" />
     <!-- Sensors -->
     <xacro:include filename="lidar.xacro" />
