Commit message: d

File: description/lidar.xacro (robot description, xacro)
@@ -1,51 +1,72 @@
 <?xml version="1.0"?>
 <robot xmlns:xacro="http://www.ros.org/wiki/xacro">
-    <!-- Lidar Joint-->
+    <!-- Fix Lidar Message type -->
+    <!-- Fix vertical sampling-->
+    <!-- Lidar Joint -->
     <joint name="lidar_joint" type="fixed">
         <parent link="chassis_link"/>
         <child link="lidar_link"/>
-        <origin xyz="0 0 -0.23" rpy="-1.570796 0 0"/> <!-- CHANGE POSITION -->
+        <origin xyz="0 0 -0.23" rpy="0 0 0"/>
     </joint>
     <!-- Lidar Link -->
     <link name="lidar_link">
         <visual>
+            <origin xyz="0 0 0" rpy="-1.578 0 0"/>
             <geometry>
-                <mesh filename="file:$(find kridtbot)/meshes/mid-360-asm(1).STL" scale="0.001 0.001 0.001"/>
+                <mesh filename="file:$(find kridtbot)/meshes/mid-360-asm.STL" scale="0.001 0.001 0.001"/>
             </geometry>
             <material name="black"/>
         </visual>
         <collision>
+            <origin xyz="0 0 0" rpy="-1.578 0 0"/>
             <geometry>
-                <mesh filename="file:$(find kridtbot)/meshes/mid-360-asm(1).STL" scale="0.001 0.001 0.001"/>
+                <mesh filename="file:$(find kridtbot)/meshes/mid-360-asm.STL" scale="0.001 0.001 0.001"/>
             </geometry>
         </collision>
     </link>
-    <!-- Gazebo tag -->
+    <!-- FOV -->
+    <link name="lidar_optical_link">
+        <visual>
+            <geometry>
+                <mesh filename="file:$(find kridtbot)/meshes/mid-360-fov-asm.STL" scale="0.0001 0.0001 0.0001"/>
+            </geometry>
+            <material name="blue opaque"/>
+        </visual>
+    </link>
+    <joint name="lidar_optical_joint" type="fixed">
+        <parent link="lidar_link"/>
+        <child link="lidar_optical_link"/>
+        <origin xyz="0 0 -0.02" rpy="-1.578 0 0"/>
+    </joint>
+    <!-- Gazebo Sensor Definition -->
     <gazebo reference="lidar_link">
         <sensor type="gpu_lidar" name="lidar_sensor">
-            <visualize>true</visualize>
+            <visualize>false</visualize>  <!-- Visualization causes crashes, disable if needed -->
             <pose>0 0 0 0 0 0</pose>
-            <update_rate>10</update_rate>
+            <update_rate>10</update_rate>  <!-- 10 Hz scan update -->
             <lidar>
+            <!-- Information from Livox specs -->
                 <scan>
                     <horizontal>
-                        <samples>360</samples>
-                        <resolution>1</resolution>
-                        <min_angle>-3.14159265359</min_angle>
-                        <max_angle>3.14159265359</max_angle>
+                        <samples>360</samples>  <!-- 360 points per rotation -->
+                        <!--<resolution>1</resolution> -->
+                        <min_angle>-3.14</min_angle>
+                        <max_angle>3.14</max_angle>
                     </horizontal>
+                    <vertical>
+                        <samples>10</samples>  <!-- 1 vertical scan -->
+                        <min_angle>0</min_angle>
+                        <max_angle>-1</max_angle>
+                    </vertical>
                 </scan>
                 <range>
-                    <min>0.3</min>
-                    <max>12</max>
+                    <min>0.1</min>  <!-- 10 cm min detection -->
+                    <max>12</max>  <!-- 70 m max detection -->
+                    <!--<resolution>0.02</resolution> -->  <!-- 2 cm precision -->
                 </range>
             </lidar>
-            <topic>scan</topic> <!-- topic to pub -->
+            <topic>lidar/points</topic>
             <gz_frame_id>lidar_link</gz_frame_id>
         </sensor>
     </gazebo>
-        <!-- Update to jazzy-->
-        <!-- change scan to mid-360 specfics-->
-        <!-- Get Gazebo control to work again-->
-        <!-- Download packages such diff_cont can activate-->
 </robot>

File: description/robot.urdf.xacro (robot description, xacro)
@@ -6,5 +6,6 @@
     <xacro:include filename="robot_core.xacro" />
     <!-- Sensors -->
-    <!-- <xacro:include filename="lidar.xacro" /> -->
+    <xacro:include filename="lidar.xacro" />
+    <xacro:include filename="depth_camera.xacro" />
     <!-- Control -->
     <xacro:if value="$(arg use_ros2_control)">

File: description/robot_core.xacro (robot description, xacro)
@@ -7,6 +7,6 @@
   <color rgba="${64/255} ${64/255} ${64/255} 1" />
 </material>
-<material name="blue">
-  <color rgba="${0/255} ${0/255} ${255/255} 1" />
+<material name="blue opaque">
+  <color rgba="${0/255} ${0/255} ${255/255} 0.4" />
 </material>
 <material name="mesh_color">
@@ -24,5 +24,5 @@
   </link>
   <joint name="base_to_chassis" type="fixed">
-    <origin xyz="0 0 0" rpy="-3.1415 0 0"/>
+    <origin xyz="0 0 0" rpy="-3.1415 0 1.57079632679"/>
     <parent link="base_link"/>
     <child link="chassis_link"/>
@@ -51,6 +51,6 @@
   <gazebo reference="chassis_link">
     <material>Gazebo/Orange</material>
-    <mu1 value = "0.3"/>
-    <mu2 value = "0.3"/>
+    <mu1 value = "1"/>
+    <mu2 value = "1"/>
   </gazebo>
     <!-- _____________BASE TO CHASSIS JOINT____________-->
@@ -117,5 +117,5 @@
     <origin xyz="0 0 -0.28" rpy="-3.1416 0 -3.1416"/>
     <axis xyz="0 0 1"/>
-    <limit effort="1000" lower="-1.5708" upper="1.5708" velocity="10"/>
+    <!--<limit effort="1000" lower="-1.5708" upper="1.5708" velocity="10"/> -->
     <parent link="diff_link"/>
     <child link="left_diff_link"/>
@@ -144,10 +144,10 @@
   <gazebo reference="left_diff_link">
     <material>Gazebo/Black</material>
-    <mu1 value = "0.3"/>
-    <mu2 value = "0.3"/>
+    <mu1 value = "1"/>
+    <mu2 value = "1"/>
   </gazebo>
   <!-- _____________LEFT DIFF TO LEFT REAR LIN JOINT____________-->
-  <joint name="left_rear_linear" type="prismatic"> <!-- left_diff_to_left_rear_lin -->
-    <limit effort="1000.0" lower="0" upper="0.13" velocity="0.5"/>
+  <joint name="left_rear_linear" type="fixed"> <!-- left_diff_to_left_rear_lin -->
+    <!--<limit effort="1000.0" lower="0" upper="0.13" velocity="0.5"/> -->
     <origin xyz="-0.216 -0.0010724 0" rpy="-1.5708 0 0.0049647"/>
     <axis xyz="0 0 1"/>
@@ -185,4 +185,5 @@
     <parent link="left_rear_lin_link"/>
     <child link="left_rear_rev_link"/>
+    <dynamics damping="0.7" friction="1"/>
   </joint>
   <!-- _____________LEFT REAR REV LINK____________-->
@@ -201,4 +202,18 @@
       </geometry>
       <material name="mesh_color"/>
+      <!--<surface>
+        <friction>
+          <ode>
+            <mu>2.0</mu>
+            <mu2>2.0</mu2>
+          </ode>
+        </friction>
+        <contact>
+          <ode>
+            <soft_cfm>0.0</soft_cfm>
+            <soft_erp>0.2</soft_erp>
+          </ode>
+        </contact>
+      </surface> -->
     </collision>
     <inertial>
@@ -209,8 +224,12 @@
   <gazebo reference="left_rear_rev_link">
     <material>Gazebo/Orange</material>
+    <mu1 value = "3"/>
+    <mu2 value = "3"/>
+    <kp>1000000.0</kp>  <!-- Contact stiffness -->
+    <kd>1.0</kd>
   </gazebo>
     <!-- _____________LEFT DIFF TO LEFT FRONT LIN JOINT____________-->
-  <joint name="left_front_linear" type="prismatic"> <!-- left_diff_to_left_front_lin-->
-    <limit effort="1000.0" lower="0" upper="0.13" velocity="0.5"/>
+  <joint name="left_front_linear" type="fixed"> <!-- left_diff_to_left_front_lin-->
+    <!--<limit effort="1000.0" lower="0" upper="0.13" velocity="0.5"/> -->
     <origin xyz="0.216 0.0010724 0" rpy="-1.5708 0 0.0049647"/>
     <axis xyz="0 0 1"/>
@@ -248,4 +267,5 @@
     <parent link="left_front_lin_link"/>
     <child link="left_front_rev_link"/>
+    <dynamics damping="0.7" friction="1"/>
   </joint>
   <!-- _____________LEFT FRONT REV LINK____________-->
@@ -264,4 +284,18 @@
       </geometry>
       <material name="mesh_color"/>
+      <!--<surface>
+        <friction>
+          <ode>
+            <mu>2.0</mu>
+            <mu2>2.0</mu2>
+          </ode>
+        </friction>
+        <contact>
+          <ode>
+            <soft_cfm>0.0</soft_cfm>
+            <soft_erp>0.2</soft_erp>
+          </ode>
+        </contact>
+      </surface> -->
     </collision>
     <inertial>
@@ -269,15 +303,19 @@
       <inertia ixx="5844491.97e-9" ixy="-376.28e-9" ixz="-3671.08e-9" iyy="5842839.83e-9" iyz="-796.72e-9" izz="3646247.90e-9"/>
     </inertial>
-    <gazebo reference="left_front_rev_link">
-      <material>Gazebo/Orange</material>
-      <mu1 value = "0.5"/>
-      <mu2 value = "0.5"/>
-    </gazebo>
-  </link>
+  </link>
+  <gazebo reference="left_front_rev_link">
+    <material>Gazebo/Black</material>
+    <mu1 value = "3"/>
+    <mu2 value = "3"/>
+    <slip1 value = "1"/>
+    <slip2 value = "1"/>
+    <kp>1000000.0</kp>  <!-- Contact stiffness -->
+    <kd>1.0</kd>
+  </gazebo>
     <!-- _____________DIFF TO RIGHT DIFF JOINT____________-->
     <joint name="right_diff" type="fixed"> <!-- diff_to_right_diff -->
       <origin xyz="0 0 0.28" rpy="0 0 0"/>
       <axis xyz="0 0 1"/>
-      <limit effort="1000" lower="-1.5708" upper="1.5708" velocity="10"/>
+      <!--<limit effort="1000" lower="-1.5708" upper="1.5708" velocity="10"/> -->
       <parent link="diff_link"/>
       <child link="right_diff_link"/>
@@ -307,11 +345,11 @@
     <gazebo reference="right_diff_link">
       <material>Gazebo/Black</material>
-      <mu1 value = "0.3"/>
-      <mu2 value = "0.3"/>
+      <mu1 value = "1"/>
+      <mu2 value = "1"/>
     </gazebo>
     <!-- _____________RIGHT DIFF TO RIGHT REAR LIN JOINT____________-->
-    <joint name="right_rear_linear" type="prismatic"> <!-- right_diff_to_right_rear_lin -->
-      <limit effort="1000.0" lower="0" upper="0.13" velocity="0.5"/>
-      <origin xyz="-0.216 -0.0010724 0" rpy="-1.5708 0 0.0049647"/>
+    <joint name="right_rear_linear" type="fixed"> <!-- right_diff_to_right_rear_lin -->
+      <!--<limit effort="1000.0" lower="0" upper="0.13" velocity="0.5"/> -->
+      <origin xyz="0.216 -0.0010724 0" rpy="-1.5708 0 0.0049647"/>
       <axis xyz="0 0 1"/>
       <parent link="right_diff_link"/>
@@ -348,4 +386,5 @@
       <parent link="right_rear_lin_link"/>
       <child link="right_rear_rev_link"/>
+      <dynamics damping="0.7" friction="1"/>
     </joint>
     <!-- _____________RIGHT REAR REV LINK____________-->
@@ -364,4 +403,18 @@
         </geometry>
         <material name="mesh_color"/>
+        <!--<surface>
+          <friction>
+            <ode>
+              <mu>2.0</mu>
+              <mu2>2.0</mu2>
+            </ode>
+          </friction>
+          <contact>
+            <ode>
+              <soft_cfm>0.0</soft_cfm>
+              <soft_erp>0.2</soft_erp>
+            </ode>
+          </contact>
+      </surface> -->
       </collision>
     <inertial>
@@ -372,9 +425,15 @@
     <gazebo reference="right_rear_rev_link">
       <material>Gazebo/Orange</material>
+      <mu1 value = "3"/>
+      <mu2 value = "3"/>
+      <slip1 value = "1"/>
+      <slip2 value = "1"/>
+      <kp>1000000.0</kp>  <!-- Contact stiffness -->
+      <kd>1.0</kd>
     </gazebo>
       <!-- _____________RIGHT DIFF TO RIGHT FRONT LIN JOINT____________-->
-    <joint name="right_front_linear" type="prismatic"> <!-- right_diff_to_right_front_lin -->
-      <limit effort="1000.0" lower="0" upper="0.13" velocity="0.5"/>
-      <origin xyz="0.216 0.0010724 0" rpy="-1.5708 0 0.0049647"/>
+    <joint name="right_front_linear" type="fixed"> <!-- right_diff_to_right_front_lin -->
+      <!--<limit effort="1000.0" lower="0" upper="0.13" velocity="0.5"/> -->
+      <origin xyz="-0.216 0.0010724 0" rpy="-1.5708 0 0.0049647"/>
       <axis xyz="0 0 1"/>
       <parent link="right_diff_link"/>
@@ -411,4 +470,5 @@
       <parent link="right_front_lin_link"/>
       <child link="right_front_rev_link"/>
+      <dynamics damping="0.7" friction="1"/>
     </joint>
     <!-- _____________RIGHT FRONT REV LINK____________-->
@@ -427,4 +487,18 @@
         </geometry>
         <material name="mesh_color"/>
+        <!--<surface>
+          <friction>
+            <ode>
+              <mu>2.0</mu>
+              <mu2>2.0</mu2>
+            </ode>
+          </friction>
+          <contact>
+            <ode>
+              <soft_cfm>0.0</soft_cfm>
+              <soft_erp>0.2</soft_erp>
+            </ode>
+          </contact>
+      </surface> -->
       </collision>
     <inertial>
@@ -435,6 +509,10 @@
     <gazebo reference="right_front_rev_link">
       <material>Gazebo/Orange</material>
-      <mu1 value = "0.5"/>
-      <mu2 value = "0.5"/>
+      <mu1 value = "3"/>
+      <mu2 value = "3"/>
+      <slip1 value = "1"/>
+      <slip2 value = "1"/>
+      <kp>1000000.0</kp>  <!-- Contact stiffness -->
+      <kd>1.0</kd>
     </gazebo>
 </robot>

Commit message: Linear_position_publishing node

File: description/lidar.xacro (robot description, xacro)
@@ -14,5 +14,5 @@
             <origin xyz="0 0 0" rpy="-1.578 0 0"/>
             <geometry>
-                <mesh filename="file:$(find kridtbot)/meshes/mid-360-asm.STL" scale="0.001 0.001 0.001"/>
+                <mesh filename="file:$(find kridtbot)/meshes/mid-360-asm.STL" scale="10.0 10.0 10.0"/>
             </geometry>
             <material name="black"/>
@@ -21,5 +21,5 @@
             <origin xyz="0 0 0" rpy="-1.578 0 0"/>
             <geometry>
-                <mesh filename="file:$(find kridtbot)/meshes/mid-360-asm.STL" scale="0.001 0.001 0.001"/>
+                <mesh filename="file:$(find kridtbot)/meshes/mid-360-asm.STL" scale="10.0 10.0 10.0"/>
             </geometry>
         </collision>
