Commit message: w

File: description/robot_sim.urdf.xacro (robot description, xacro)
@@ -4,5 +4,5 @@
     <xacro:arg name="use_ros2_control" default="true"/>
     <!-- URDF Robot Description-->
-    <xacro:include filename="robot_core_sim.xacro" />
+    <xacro:include filename="robot_core.xacro" />
     <!-- Sensors -->
     <xacro:include filename="lidar.xacro" />
@@ -10,5 +10,6 @@
     <!-- Control -->
     <xacro:if value="$(arg use_ros2_control)">
-        <xacro:include filename="ros2_control_gz.xacro" />
+        <xacro:include filename="ros2_control_gz_myactuator.xacro" />
+        <!--<xacro:include filename="ros2_control_gz_odrive.xacro" /> -->
     </xacro:if>
     <xacro:unless value="$(arg use_ros2_control)">

File: description/ros2_control_gz_myactuator.xacro (robot description, xacro)
@@ -2,5 +2,5 @@
 <robot xmlns:xacro="http://www.ros.org/wiki/xacro">
     <!-- ROS2 Control plugin for Gazebo-->
-    <ros2_control name="GazeboSystem" type="system">
+    <ros2_control name="GazeboSystemMyActuator" type="system">
         <!-- Hardware interface for GZ-->
         <hardware>
@@ -28,4 +28,37 @@
             <state_interface name="position"></state_interface>
         </joint>
+        <!-- All prismatic joints -->
+        <joint name="right_rear_linear">
+            <command_interface name="position"/>
+            <command_interface name="velocity"/>
+            <command_interface name="effort"/>
+            <state_interface name="position"/>
+            <state_interface name="velocity"/>
+            <state_interface name="effort"/>
+        </joint>
+        <joint name="right_front_linear">
+            <command_interface name="position"/>
+            <command_interface name="velocity"/>
+            <command_interface name="effort"/>
+            <state_interface name="position"/>
+            <state_interface name="velocity"/>
+            <state_interface name="effort"/>
+        </joint>
+        <joint name="left_rear_linear">
+            <command_interface name="position"/>
+            <command_interface name="velocity"/>
+            <command_interface name="effort"/>
+            <state_interface name="position"/>
+            <state_interface name="velocity"/>
+            <state_interface name="effort"/>
+        </joint>
+        <joint name="left_front_linear">
+            <command_interface name="position"/>
+            <command_interface name="velocity"/>
+            <command_interface name="effort"/>
+            <state_interface name="position"/>
+            <state_interface name="velocity"/>
+            <state_interface name="effort"/>
+        </joint>
     </ros2_control>
         <!-- GZ plugin -->

File: description/ros2_control_gz_odrive.xacro (robot description, xacro)
@@ -2,11 +2,11 @@
 <robot xmlns:xacro="http://www.ros.org/wiki/xacro">
     <!-- ROS2 Control plugin for Gazebo-->
-    <ros2_control name="odrive_controller" type="system">
+    <ros2_control name="GazeboSystemODrive" type="system">
+        <!-- Hardware interface for GZ-->
         <hardware>
-            <plugin>odrive_ros2_control_plugin/ODriveHardwareInterface</plugin>
-            <param name="can">can4</param>
+            <plugin>gz_ros2_control/GazeboSimSystem</plugin>
         </hardware>
+        <!-- All continous joints-->
         <joint name="right_rear_linear">
-            <param name="node_id">3</param>
             <command_interface name="position"/>
             <command_interface name="velocity"/>
@@ -17,6 +17,5 @@
         </joint>
         <joint name="right_front_linear">
-            <param name="node_id">2</param>
-        ->  <command_interface name="position"/>
+            <command_interface name="position"/>
             <command_interface name="velocity"/>
             <command_interface name="effort"/>
@@ -26,5 +25,4 @@
         </joint>
         <joint name="left_rear_linear">
-            <param name="node_id">1</param>
             <command_interface name="position"/>
             <command_interface name="velocity"/>
@@ -35,5 +33,4 @@
         </joint>
         <joint name="left_front_linear">
-            <param name="node_id">0</param>
             <command_interface name="position"/>
             <command_interface name="velocity"/>
@@ -44,3 +41,9 @@
         </joint>
     </ros2_control>
+        <!-- GZ plugin -->
+    <gazebo>
+          <plugin name="gz_ros2_control::GazeboSimROS2ControlPlugin" filename="libgz_ros2_control-system.so">
+            <parameters>$(find kridtbot)/config/my_controllers.yaml</parameters>
+        </plugin>
+    </gazebo>
 </robot>
