Commit message: d

File: description/robot_core.xacro (robot description, xacro)
@@ -182,5 +182,5 @@
   </gazebo>
     <!-- _____________LEFT DIFF TO LEFT FRONT LIN JOINT____________-->
-  <joint name="left_front_linear" type="fixed"> <!-- left_diff_to_left_front_lin-->
+  <joint name="left_front_linear" type="prismatic"> <!-- left_diff_to_left_front_lin-->
     <limit effort="1000.0" lower="0" upper="0.13" velocity="0.5"/>
     <origin xyz="0.216 0.0010724 0" rpy="-1.5708 0 0.0049647"/>
@@ -282,5 +282,5 @@
     </gazebo>
     <!-- _____________RIGHT DIFF TO RIGHT REAR LIN JOINT____________-->
-    <joint name="right_rear_linear" type="fixed"> <!-- right_diff_to_right_rear_lin -->
+    <joint name="right_rear_linear" type="prismatic"> <!-- right_diff_to_right_rear_lin -->
       <limit effort="1000.0" lower="0" upper="0.13" velocity="0.5"/>
       <origin xyz="-0.216 -0.0010724 0" rpy="-1.5708 0 0.0049647"/>
@@ -345,5 +345,5 @@
     </gazebo>
       <!-- _____________RIGHT DIFF TO RIGHT FRONT LIN JOINT____________-->
-    <joint name="right_front_linear" type="fixed"> <!-- right_diff_to_right_front_lin -->
+    <joint name="right_front_linear" type="prismatic"> <!-- right_diff_to_right_front_lin -->
       <limit effort="1000.0" lower="0" upper="0.13" velocity="0.5"/>
       <origin xyz="0.216 0.0010724 0" rpy="-1.5708 0 0.0049647"/>

Commit message: d

File: description/robot_core.xacro (robot description, xacro)
@@ -84,4 +84,33 @@
     <material>Gazebo/Orange</material>
   </gazebo>
+  <link name="imu_link">
+    <visual>
+      <origin xyz="-0.028 -0.019 -0.01" rpy="1.57079633 0 1.57079633"/>
+      <geometry>
+        <mesh filename="file:$(find kridtbot)/meshes/imu_link.STL"/>
+      </geometry>
+      <material name = "black"/>
+    </visual>
+    <collision>
+      <origin xyz="0 0 0" rpy="0 0 0"/>
+      <geometry>
+        <mesh filename="file:$(find kridtbot)/meshes/imu_link.STL"/>
+      </geometry>
+      <material name="mesh_color"/>
+    </collision>
+    <inertial>
+      <mass value="0.02302"/>
+      <inertia ixx="3763.33e-9" ixy="0" ixz="0" iyy="6942.61e-9" iyz="0" izz="9041.46e-9"/>
+    </inertial>
+  </link>
+  <!-- _____________DIFF TO IMU JOINT____________-->
+  <joint name="diff_to_imu" type="fixed">
+    <origin xyz="0 -0.038 0" rpy="1.57079633 3.14159265 0"/>
+    <parent link="diff_link"/>
+    <child link="imu_link"/>
+  </joint>
+  <gazebo reference="imu_link">
+    <material>Gazebo/Black</material>
+  </gazebo>
   <!-- _____________DIFF TO LEFT DIFF JOINT____________-->
   <joint name="left_diff" type="fixed"> <!--diff_to_left_diff-->

Commit message: d

File: description/robot_core.xacro (robot description, xacro)
@@ -149,5 +149,5 @@
   <!-- _____________LEFT DIFF TO LEFT REAR LIN JOINT____________-->
   <joint name="left_rear_linear" type="prismatic"> <!-- left_diff_to_left_rear_lin -->
-    <!--<limit effort="1000.0" lower="0" upper="0.13" velocity="0.5"/> -->
+    <limit effort="1000.0" lower="0" upper="0.13" velocity="0.5"/>
     <origin xyz="-0.216 -0.0010724 0" rpy="-1.5708 0 0.0049647"/>
     <axis xyz="0 0 1"/>
@@ -231,5 +231,5 @@
     <!-- _____________LEFT DIFF TO LEFT FRONT LIN JOINT____________-->
   <joint name="left_front_linear" type="prismatic"> <!-- left_diff_to_left_front_lin-->
-    <!--<limit effort="1000.0" lower="0" upper="0.13" velocity="0.5"/> -->
+    <limit effort="1000.0" lower="0" upper="0.13" velocity="0.5"/>
     <origin xyz="0.216 0.0010724 0" rpy="-1.5708 0 0.0049647"/>
     <axis xyz="0 0 1"/>
@@ -350,5 +350,5 @@
     <!-- _____________RIGHT DIFF TO RIGHT REAR LIN JOINT____________-->
     <joint name="right_rear_linear" type="prismatic"> <!-- right_diff_to_right_rear_lin -->
-      <!--<limit effort="1000.0" lower="0" upper="0.13" velocity="0.5"/> -->
+      <limit effort="1000.0" lower="0" upper="0.13" velocity="0.5"/>
       <origin xyz="0.216 -0.0010724 0" rpy="-1.5708 0 0.0049647"/>
       <axis xyz="0 0 1"/>
@@ -434,5 +434,5 @@
       <!-- _____________RIGHT DIFF TO RIGHT FRONT LIN JOINT____________-->
     <joint name="right_front_linear" type="prismatic"> <!-- right_diff_to_right_front_lin -->
-      <!--<limit effort="1000.0" lower="0" upper="0.13" velocity="0.5"/> -->
+      <limit effort="1000.0" lower="0" upper="0.13" velocity="0.5"/>
       <origin xyz="-0.216 0.0010724 0" rpy="-1.5708 0 0.0049647"/>
       <axis xyz="0 0 1"/>

Commit message: w

File: description/robot_core.xacro (robot description, xacro)
@@ -1,19 +1,19 @@
 <?xml version="1.0"?>
 <robot xmlns:xacro="http://www.ros.org/wiki/xacro">
-<material name="orange">
-  <color rgba="${252/255} ${188/255} ${132/255} 1" />
-</material>
-<material name="black">
-  <color rgba="${64/255} ${64/255} ${64/255} 1" />
-</material>
-<material name="blue opaque">
-  <color rgba="${0/255} ${0/255} ${255/255} 0.4" />
-</material>
-<material name="mesh_color">
-  <color rgba="${0/255} ${0/255} ${255/255} 0.6" />
-</material>
+  <!-- Materials -->
+  <material name="orange">
+    <color rgba="${252/255} ${188/255} ${132/255} 1" />
+  </material>
+  <material name="black">
+    <color rgba="${64/255} ${64/255} ${64/255} 1" />
+  </material>
+  <material name="blue opaque">
+    <color rgba="${0/255} ${0/255} ${255/255} 0.4" />
+  </material>
+  <material name="mesh_color">
+    <color rgba="${0/255} ${0/255} ${255/255} 0.6" />
+  </material>
   <!-- ________BASE LINK__________-->
-  <link name="base_link">
-  </link>
+  <link name="base_link" />
   <joint name="base_footprint_joint" type="fixed">
     <origin xyz="0 0 0" rpy="0 0 0"/>
@@ -21,6 +21,5 @@
     <child link="base_footprint"/>
   </joint>
-  <link name="base_footprint">
-  </link>
+  <link name="base_footprint" />
   <joint name="base_to_chassis" type="fixed">
     <origin xyz="0 0 0" rpy="-3.1415 0 1.57079632679"/>
@@ -46,13 +45,13 @@
     <inertial>
       <mass value="11.18100"/>
-      <inertia ixx="0.52" ixy=" 0.00" ixz="0.00" iyy="0.48" iyz=" 0.04" izz="0.60"/>
+      <inertia ixx="0.52" ixy="0.00" ixz="0.00" iyy="0.48" iyz="0.04" izz="0.60"/>
     </inertial>
   </link>
   <gazebo reference="chassis_link">
     <material>Gazebo/Orange</material>
-    <mu1 value = "1"/>
-    <mu2 value = "1"/>
-  </gazebo>
-    <!-- _____________BASE TO CHASSIS JOINT____________-->
+    <mu1 value="1"/>
+    <mu2 value="1"/>
+  </gazebo>
+  <!-- _____________DIFF LINK____________-->
   <joint name="chassis_to_diff" type="fixed">
     <origin xyz="-0.00062572 0.016893 -0.01406" rpy="1.5708 0 -1.5708"/>
@@ -60,5 +59,4 @@
     <child link="diff_link"/>
   </joint>
-  <!-- _____________DIFF LINK____________-->
   <link name="diff_link">
     <visual>
@@ -67,5 +65,5 @@
         <mesh filename="file:$(find kridtbot)/meshes/diff_link.STL"/>
       </geometry>
-      <material name = "black"/>
+      <material name="black"/>
     </visual>
     <collision>
@@ -78,48 +76,27 @@
     <inertial>
       <mass value="1.44"/>
-      <inertia ixx="2024193.31e-9" ixy="258.53e-9" ixz="-42.56e-9" iyy="1553917.67e-9" iyz=" 559.93e-9" izz="1298088.14e-9"/>
+      <inertia ixx="2024193.31e-9" ixy="258.53e-9" ixz="-42.56e-9" iyy="1553917.67e-9" iyz="559.93e-9" izz="1298088.14e-9"/>
     </inertial>
   </link>
   <gazebo reference="diff_link">
     <material>Gazebo/Orange</material>
-  </gazebo>
-  <link name="imu_link">
-    <visual>
-      <origin xyz="-0.028 -0.019 -0.01" rpy="1.57079633 0 1.57079633"/>
-      <geometry>
-        <mesh filename="file:$(find kridtbot)/meshes/imu_link.STL"/>
-      </geometry>
-      <material name = "black"/>
-    </visual>
-    <collision>
-      <origin xyz="0 0 0" rpy="0 0 0"/>
-      <geometry>
-        <mesh filename="file:$(find kridtbot)/meshes/imu_link.STL"/>
-      </geometry>
-      <material name="mesh_color"/>
-    </collision>
-    <inertial>
-      <mass value="0.02302"/>
-      <inertia ixx="3763.33e-9" ixy="0" ixz="0" iyy="6942.61e-9" iyz="0" izz="9041.46e-9"/>
-    </inertial>
-  </link>
-  <!-- _____________DIFF TO IMU JOINT____________-->
-  <joint name="diff_to_imu" type="fixed">
-    <origin xyz="0 -0.038 0" rpy="1.57079633 3.14159265 0"/>
-    <parent link="diff_link"/>
-    <child link="imu_link"/>
-  </joint>
-  <gazebo reference="imu_link">
-    <material>Gazebo/Black</material>
-  </gazebo>
-  <!-- _____________DIFF TO LEFT DIFF JOINT____________-->
-  <joint name="left_diff" type="fixed"> <!--diff_to_left_diff-->
+    <mu1 value="1"/>
+    <mu2 value="1"/>
+  </gazebo>
+  <!-- _____________ 1. LEFT DIFF LINK ____________-->
+  <joint name="left_diff" type="continuous">
     <origin xyz="0 0 -0.28" rpy="-3.1416 0 -3.1416"/>
     <axis xyz="0 0 1"/>
-    <!--<limit effort="1000" lower="-1.5708" upper="1.5708" velocity="10"/> -->
     <parent link="diff_link"/>
     <child link="left_diff_link"/>
-  </joint>
-  <!-- _____________LEFT DIFF LINK____________-->
+    <!--<mimic joint="center_diff" multiplier="1" offset="0"/> -->
+  </joint>
+  <gazebo reference="left_diff">
+    <material>Gazebo/Black</material>
+    <mu1 value="1000"/>
+    <mu2 value="1000"/>
+    <provideFeedback>true</provideFeedback>
+    <implicitSpringDamper>true</implicitSpringDamper>
+  </gazebo>
   <link name="left_diff_link">
     <visual>
@@ -128,5 +105,5 @@
         <mesh filename="file:$(find kridtbot)/meshes/left_diff_link.STL"/>
       </geometry>
-      <material name = "black"/>
+      <material name="black"/>
     </visual>
     <collision>
@@ -144,9 +121,9 @@
   <gazebo reference="left_diff_link">
     <material>Gazebo/Black</material>
-    <mu1 value = "1"/>
-    <mu2 value = "1"/>
-  </gazebo>
-  <!-- _____________LEFT DIFF TO LEFT REAR LIN JOINT____________-->
-  <joint name="left_rear_linear" type="prismatic"> <!-- left_diff_to_left_rear_lin -->
+    <mu1 value="1"/>
+    <mu2 value="1"/>
+  </gazebo>
+  <!-- _____________LEFT REAR LINEAR ACtuator____________-->
+  <joint name="left_rear_linear" type="prismatic">
     <limit effort="1000.0" lower="0" upper="0.13" velocity="0.5"/>
     <origin xyz="-0.216 -0.0010724 0" rpy="-1.5708 0 0.0049647"/>
@@ -155,5 +132,4 @@
     <child link="left_rear_lin_link"/>
   </joint>
-  <!-- _____________LEFT REAR LIN LINK____________-->
   <link name="left_rear_lin_link">
     <visual>
@@ -162,5 +138,5 @@
         <mesh filename="file:$(find kridtbot)/meshes/left_rear_lin_link.STL"/>
       </geometry>
-      <material name = "black"/>
+      <material name="black"/>
     </visual>
     <collision>
@@ -173,5 +149,5 @@
     <inertial>
       <mass value="1.04456"/>
-      <inertia ixx="59743728.97e-9" ixy="-5941.33e-9" ixz="293509.06e-9" iyy="59856745.28e-9" iyz=" -1015856.43e-9" izz="595093.96e-9"/>
+      <inertia ixx="59743728.97e-9" ixy="-5941.33e-9" ixz="293509.06e-9" iyy="59856745.28e-9" iyz="-1015856.43e-9" izz="595093.96e-9"/>
     </inertial>
   </link>
@@ -179,6 +155,6 @@
     <material>Gazebo/Black</material>
   </gazebo>
-<!-- _____________LEFT REAR LIN TO LEFT REAR REV JOINT____________-->
-  <joint name="left_rear_wheel" type="continuous"> <!-- left_rear_lin_to_left_rear_rev -->
+  <!-- _____________LEFT REAR wheel ____________-->
+  <joint name="left_rear_wheel" type="continuous">
     <origin xyz="0.0012158 0 0.2449" rpy="1.5708 0 0"/>
     <axis xyz="0 0 1"/>
@@ -187,5 +163,4 @@
     <dynamics damping="0.7" friction="1"/>
   </joint>
-  <!-- _____________LEFT REAR REV LINK____________-->
   <link name="left_rear_rev_link">
     <visual>
@@ -194,26 +169,12 @@
         <cylinder radius="0.0865" length="0.05234"/>
       </geometry>
-      <material name = "orange"/>
-    </visual>
-    <collision>
-      <origin xyz="0 0 0.06266" rpy="0 0 0"/>
-      <geometry>
-        <cylinder radius="0.0865" length="0.05234"/>
-      </geometry>
-      <material name="mesh_color"/>
-      <!--<surface>
-        <friction>
-          <ode>
-            <mu>2.0</mu>
-            <mu2>2.0</mu2>
-          </ode>
-        </friction>
-        <contact>
-          <ode>
-            <soft_cfm>0.0</soft_cfm>
-            <soft_erp>0.2</soft_erp>
-          </ode>
-        </contact>
-      </surface> -->
+      <material name="orange"/>
+    </visual>
+    <collision>
+      <origin xyz="0 0 0.06266" rpy="0 0 0"/>
+      <geometry>
+        <cylinder radius="0.0865" length="0.05234"/>
+      </geometry>
+      <material name="mesh_color"/>
     </collision>
     <inertial>
@@ -224,11 +185,11 @@
   <gazebo reference="left_rear_rev_link">
     <material>Gazebo/Orange</material>
-    <mu1 value = "3"/>
-    <mu2 value = "3"/>
-    <kp>1000000.0</kp>  <!-- Contact stiffness -->
+    <mu1 value="3"/>
+    <mu2 value="3"/>
+    <kp>1000000.0</kp>
     <kd>1.0</kd>
   </gazebo>
-    <!-- _____________LEFT DIFF TO LEFT FRONT LIN JOINT____________-->
-  <joint name="left_front_linear" type="prismatic"> <!-- left_diff_to_left_front_lin-->
+  <!-- _____________LEFT FRONT LINEAR actuator____________-->
+  <joint name="left_front_linear" type="prismatic">
     <limit effort="1000.0" lower="0" upper="0.13" velocity="0.5"/>
     <origin xyz="0.216 0.0010724 0" rpy="-1.5708 0 0.0049647"/>
@@ -237,5 +198,4 @@
     <child link="left_front_lin_link"/>
   </joint>
-  <!-- _____________LEFT FRONT LIN LINK____________-->
   <link name="left_front_lin_link">
     <visual>
@@ -244,5 +204,5 @@
         <mesh filename="file:$(find kridtbot)/meshes/front_left_lin_link.STL"/>
       </geometry>
-      <material name = "black"/>
+      <material name="black"/>
     </visual>
     <collision>
@@ -255,12 +215,12 @@
     <inertial>
       <mass value="1.04456"/>
-      <inertia ixx="59743728.97e-9" ixy="-5941.33e-9" ixz="293509.06e-9" iyy="59856745.28e-9" iyz=" -1015856.43e-9" izz="595093.96e-9"/>
-    </inertial>
-  </link>
-  <gazebo reference="left_front_lin_link"> <!-- left_front_link_link-->
-    <material>Gazebo/Black</material>
-  </gazebo>
-<!-- _____________LEFT FRONT LIN TO LEFT FRONT REV JOINT____________-->
-  <joint name="left_front_wheel" type="continuous"> <!-- left_front_lin_to_left_front_rev -->
+      <inertia ixx="59743728.97e-9" ixy="-5941.33e-9" ixz="293509.06e-9" iyy="59856745.28e-9" iyz="-1015856.43e-9" izz="595093.96e-9"/>
+    </inertial>
+  </link>
+  <gazebo reference="left_front_lin_link">
+    <material>Gazebo/Black</material>
+  </gazebo>
+  <!-- _____________LEFT FRONT wheel ____________-->
+  <joint name="left_front_wheel" type="continuous">
     <origin xyz="0.0012158 0 0.2449" rpy="1.5708 0 0"/>
     <axis xyz="0 0 1"/>
@@ -269,5 +229,4 @@
     <dynamics damping="0.7" friction="1"/>
   </joint>
-  <!-- _____________LEFT FRONT REV LINK____________-->
   <link name="left_front_rev_link">
     <visual>
@@ -276,26 +235,12 @@
         <cylinder radius="0.0865" length="0.05234"/>
       </geometry>
-      <material name = "orange"/>
-    </visual>
-    <collision>
-      <origin xyz="0 0 0.06266" rpy="0 0 0"/>
-      <geometry>
-        <cylinder radius="0.0865" length="0.05234"/>
-      </geometry>
-      <material name="mesh_color"/>
-      <!--<surface>
-        <friction>
-          <ode>
-            <mu>2.0</mu>
-            <mu2>2.0</mu2>
-          </ode>
-        </friction>
-        <contact>
-          <ode>
-            <soft_cfm>0.0</soft_cfm>
-            <soft_erp>0.2</soft_erp>
-          </ode>
-        </contact>
-      </surface> -->
+      <material name="orange"/>
+    </visual>
+    <collision>
+      <origin xyz="0 0 0.06266" rpy="0 0 0"/>
+      <geometry>
+        <cylinder radius="0.0865" length="0.05234"/>
+      </geometry>
+      <material name="mesh_color"/>
     </collision>
     <inertial>
@@ -306,213 +251,212 @@
   <gazebo reference="left_front_rev_link">
     <material>Gazebo/Black</material>
-    <mu1 value = "3"/>
-    <mu2 value = "3"/>
-    <slip1 value = "1"/>
-    <slip2 value = "1"/>
-    <kp>1000000.0</kp>  <!-- Contact stiffness -->
+    <mu1 value="3"/>
+    <mu2 value="3"/>
+    <slip1 value="1"/>
+    <slip2 value="1"/>
+    <kp>1000000.0</kp>
     <kd>1.0</kd>
   </gazebo>
-    <!-- _____________DIFF TO RIGHT DIFF JOINT____________-->
-    <joint name="right_diff" type="fixed"> <!-- diff_to_right_diff -->
-      <origin xyz="0 0 0.28" rpy="0 0 0"/>
-      <axis xyz="0 0 1"/>
-      <!--<limit effort="1000" lower="-1.5708" upper="1.5708" velocity="10"/> -->
-      <parent link="diff_link"/>
-      <child link="right_diff_link"/>
-      <mimic joint="left_diff" multiplier="1"/>
-    </joint>
-    <!-- _____________RIGHT DIFF LINK____________-->
-    <link name="right_diff_link">
-      <visual>
-        <origin xyz="0 0 0" rpy="0 0 0"/>
-        <geometry>
-          <mesh filename="file:$(find kridtbot)/meshes/rigth_diff_link.STL"/>
-        </geometry>
-        <material name = "black"/>
-      </visual>
-      <collision>
-        <origin xyz="0 0 0" rpy="0 0 0"/>
-        <geometry>
-          <mesh filename="file:$(find kridtbot)/meshes/rigth_diff_link.STL"/>
-        </geometry>
-        <material name="mesh_color"/>
-      </collision>
+  <!-- _____________ 2. RIGHT DIFF LINK____________-->
+  <joint name="right_diff" type="continuous">
+    <origin xyz="0 0 0.28" rpy="0 0 0"/>
+    <axis xyz="0 0 1"/>
+    <parent link="diff_link"/>
+    <child link="right_diff_link"/>
+    <!--<mimic joint="center_diff" multiplier="-1" offset="0"/>-->
+  </joint>
+  <link name="right_diff_link">
+    <visual>
+      <origin xyz="0 0 0" rpy="0 0 0"/>
+      <geometry>
+        <mesh filename="file:$(find kridtbot)/meshes/rigth_diff_link.STL"/>
+      </geometry>
+      <material name="black"/>
+    </visual>
+    <collision>
+      <origin xyz="0 0 0" rpy="0 0 0"/>
+      <geometry>
+        <mesh filename="file:$(find kridtbot)/meshes/rigth_diff_link.STL"/>
+      </geometry>
+      <material name="mesh_color"/>
+    </collision>
     <inertial>
       <mass value="7.30200"/>
       <inertia ixx="133810688.94e-9" ixy="319399.82e-9" ixz="2255.98e-9" iyy="282053860.06e-9" iyz="-558.22e-9" izz="397597733.07e-9"/>
     </inertial>
-    </link>
-    <gazebo reference="right_diff_link">
-      <material>Gazebo/Black</material>
-      <mu1 value = "1"/>
-      <mu2 value = "1"/>
-    </gazebo>
-    <!-- _____________RIGHT DIFF TO RIGHT REAR LIN JOINT____________-->
-    <joint name="right_rear_linear" type="prismatic"> <!-- right_diff_to_right_rear_lin -->
-      <limit effort="1000.0" lower="0" upper="0.13" velocity="0.5"/>
-      <origin xyz="0.216 -0.0010724 0" rpy="-1.5708 0 0.0049647"/>
-      <axis xyz="0 0 1"/>
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
File: description/robot_sim.urdf.xacro (robot description, xacro)
@@ -8,8 +8,8 @@
     <xacro:include filename="lidar.xacro" />
     <xacro:include filename="depth_camera.xacro" />
+    <xacro:include filename="imu.xacro" />
     <!-- Control -->
     <xacro:if value="$(arg use_ros2_control)">
-        <xacro:include filename="ros2_control_gz_myactuator.xacro" />
-        <!--<xacro:include filename="ros2_control_gz_odrive.xacro" /> -->
+        <xacro:include filename="ros2_control_gz.xacro" />
     </xacro:if>
     <xacro:unless value="$(arg use_ros2_control)">

File: description/ros2_control_gz.xacro (robot description, xacro)
@@ -2,5 +2,5 @@
 <robot xmlns:xacro="http://www.ros.org/wiki/xacro">
     <!-- ROS2 Control plugin for Gazebo-->
-    <ros2_control name="GazeboSystemMyActuator" type="system">
+    <ros2_control name="GazeboSystem" type="system">
         <!-- Hardware interface for GZ-->
         <hardware>
@@ -61,5 +61,37 @@
             <state_interface name="effort"/>
         </joint>
+        <!-- IMU sensor-->
+        <sensor name="imu_sensor">
+            <param name="frame_id">imu_link</param>
+            <state_interface name="orientation.x"/>
+            <state_interface name="orientation.y"/>
+            <state_interface name="orientation.z"/>
+            <state_interface name="orientation.w"/>
+            <state_interface name="angular_velocity.x"/>
+            <state_interface name="angular_velocity.y"/>
+            <state_interface name="angular_velocity.z"/>
+            <state_interface name="linear_acceleration.x"/>
+            <state_interface name="linear_acceleration.y"/>
+            <state_interface name="linear_acceleration.z"/>
+        </sensor>
     </ros2_control>
+   <!-- <ros2_control name="imu_broad" type="sensor">
+        <hardware>
+            <plugin>gazebo_ros2_control/GazeboSensorSystem</plugin>
+        </hardware>
+        <sensor name="imu_sensor">
+                <param name="frame_id">imu_link</param>
+                <state_interface name="orientation.x" />
+                <state_interface name="orientation.y" />
+                <state_interface name="orientation.z" />
+                <state_interface name="orientation.w" />
+                <state_interface name="angular_velocity.x" />
+                <state_interface name="angular_velocity.y" />
+                <state_interface name="angular_velocity.z" />
+                <state_interface name="linear_acceleration.x" />
+                <state_interface name="linear_acceleration.y" />
+                <state_interface name="linear_acceleration.z" />
+            </sensor>
+        </ros2_control> -->
         <!-- GZ plugin -->
     <gazebo>
